Commit message: default

File: description/robot_core.xacro (robot description, xacro)
@@ -16,4 +16,5 @@
     <link name="base_link">
     </link>
+    <!-- CHASSIS LINK -->
     <joint name= "chassis_joint" type = "fixed">
         <parent link="base_link"/>
@@ -30,3 +31,16 @@
          </visual>
     </link>
+    <!--LEFT WHEEL LINK-->
+    <joint name='left_wheel_joint' type='continuos'>
+        <parent link = 'base_link'/>
+        <child link='left_wheel'/>
+    </joint>
+    <link name = 'left_wheel'>
+        <visual>
+            <geometry>
+                <cylinder radius='.05' length='0.04'/>
+            </geometry>
+            <material name='blue'/>
+        </visual>
+    </link>
 </robot>

Commit message: inertial file and complete setup for physical base

File: description/robot_core.xacro (robot description, xacro)
@@ -1,4 +1,5 @@
 <?xml version="1.0"?>
-<robot xmlns:xacro="http://www.ros.org/wiki/xacro"  >
+<robot xmlns:xacro="http://www.ros.org/wiki/xacro">
+    <xacro:include filename='inertial_macros.xacro'/>
     <material name="white">
         <color rgba = "1 1 1 1"/>
@@ -8,5 +9,5 @@
     </material>
     <material name="blue">
-        <color rgba="1 0.3 0.1 1" />
+        <color rgba=".2 .2 1 1" />
     </material>
     <material name="black">
@@ -20,5 +21,5 @@
         <parent link="base_link"/>
         <child link="chassis"/>
-        <origin xyz="-0.1 0 0"/>
+        <origin xyz="0.01 0 0"/>
     </joint>
     <link name ="chassis">
@@ -26,21 +27,107 @@
             <origin xyz="0.15 0 0.075"/>
             <geometry>
-                <box size="0.3 0.3 0.15"/>
+                <box size="0.5 0.3 0.15"/>
             </geometry>
             <material name="white"/>
-         </visual>
+        </visual>
+        <collision>
+            <origin xyz="0.15 0 0.075"/>
+            <geometry>
+                <box size="0.5 0.3 0.15"/>
+            </geometry>
+        </collision>
+        <xacro:inertial_box mass = '.5' x='.3' y='.3' z='.15'>
+            <origin xyz='.15' '0' '0' '.75' rpy='0 0 0'/>
+        </xacro:inertial_box>
     </link>
     <!--LEFT WHEEL LINK-->
-    <joint name='left_wheel_joint' type='continuos'>
+    <joint name='left_wheel_joint' type='continuous'>
         <parent link = 'base_link'/>
         <child link='left_wheel'/>
+        <origin xyz = '0 0.175 0' rpy = '-${pi/2} 0 0'/>
+        <axis xyz = '0 0 1'/>
     </joint>
     <link name = 'left_wheel'>
         <visual>
             <geometry>
-                <cylinder radius='.05' length='0.04'/>
+                <cylinder radius='0.05' length='0.04'/>
             </geometry>
             <material name='blue'/>
         </visual>
+        <collision>
+            <geometry>
+                <cylinder radius='0.05' length='0.04'/>
+            </geometry>
+        </collision>
+        <xacro:inertial_cylinder mass='.1' length='.04' radius='.05'>
+            <origin xyz='0 0 0' rpy='0 0 0'/>
+        </xacro:inertial_cylinder>
+    </link>
+    <!--RIGHT WHEEL LINK-->
+    <joint name='right_wheel_joint' type='continuous'>
+        <parent link = 'base_link'/>
+        <child link='right_wheel'/>
+        <origin xyz = '0 -0.175 0' rpy = '${pi/2} 0 0'/>
+        <axis xyz = '0 0 -1'/>
+    </joint>
+    <link name = 'right_wheel'>
+        <visual>
+            <geometry>
+                <cylinder radius='0.05' length='0.04'/>
+            </geometry>
+            <material name='blue'/>
+        </visual>
+        <collision>
+            <geometry>
+                <cylinder radius='0.05' length='0.04'/>
+            </geometry>
+        </collision>
+        <xacro:inertial_cylinder mass='.1' length='.04' radius='.05'>
+            <origin xyz='0 0 0' rpy='0 0 0'/>
+        </xacro:inertial_cylinder>
+    </link>
+    <!--LEFT CASTER WHEEL LINK-->
+    <joint name='L_caster_wheel_joint' type = 'fixed'>
+        <parent link='base_link'/>
+        <child link='L_caster_wheel'/>
+        <origin xyz = '0.24 0.175 0' rpy = '-${pi/2} 0 0'/>
+    </joint>
+    <link name = 'L_caster_wheel'>
+        <visual>
+            <geometry>
+                <cylinder radius = '0.05' length ='0.04'/>
+            </geometry>
+            <material name = 'black'/>
+        </visual>
+        <collision>
+            <geometry>
+                <cylinder radius = '0.05' length ='0.04'/>
+            </geometry>
+        </collision>
+        <xacro:inertial_cylinder mass='.1' length='.04' radius='.05'>
+            <origin xyz='0 0 0' rpy='0 0 0'/>
+        </xacro:inertial_cylinder>
+    </link>
+        <!--RIGHT CASTER WHEEL LINK-->
+    <joint name='R_caster_wheel_joint' type = 'fixed'>
+        <parent link='base_link'/>
+        <child link='R_caster_wheel'/>
+        <origin xyz = '0.24 -0.175 0' rpy = '${pi/2} 0 0'/>
+    </joint>
+    <link name = 'R_caster_wheel'>
+        <visual>
+            <geometry>
+                <cylinder radius = '0.05' length ='0.04'/>
+            </geometry>
+            <material name = 'black'/>
+        </visual>
+        <collision>
+            <geometry>
+                <cylinder radius = '0.05' length ='0.04'/>
+            </geometry>
+        </collision>
+        <xacro:inertial_cylinder mass='.1' length='.04' radius='.05'>
+            <origin xyz='0 0 0' rpy='0 0 0'/>
+        </xacro:inertial_cylinder>
     </link>
 </robot>

Commit message: finished setup xrdf file

File: description/robot_core.xacro (robot description, xacro)
@@ -1,5 +1,5 @@
 <?xml version="1.0"?>
 <robot xmlns:xacro="http://www.ros.org/wiki/xacro">
-    <xacro:include filename='inertial_macros.xacro'/>
+    <xacro:include filename="inertial_macros.xacro"/>
     <material name="white">
         <color rgba = "1 1 1 1"/>
@@ -37,6 +37,6 @@
             </geometry>
         </collision>
-        <xacro:inertial_box mass = '.5' x='.3' y='.3' z='.15'>
-            <origin xyz='.15' '0' '0' '.75' rpy='0 0 0'/>
+        <xacro:inertial_box mass = "0.5" x="0.3" y="0.3" z="0.15">
+            <origin xyz="0.15 0 0.75" rpy="0 0 0"/>
         </xacro:inertial_box>
     </link>
@@ -60,5 +60,5 @@
             </geometry>
         </collision>
-        <xacro:inertial_cylinder mass='.1' length='.04' radius='.05'>
+        <xacro:inertial_cylinder mass='0.1' length='.04' radius='.05'>
             <origin xyz='0 0 0' rpy='0 0 0'/>
         </xacro:inertial_cylinder>
@@ -83,5 +83,5 @@
             </geometry>
         </collision>
-        <xacro:inertial_cylinder mass='.1' length='.04' radius='.05'>
+        <xacro:inertial_cylinder mass='0.1' length='.04' radius='.05'>
             <origin xyz='0 0 0' rpy='0 0 0'/>
         </xacro:inertial_cylinder>
@@ -105,5 +105,5 @@
             </geometry>
         </collision>
-        <xacro:inertial_cylinder mass='.1' length='.04' radius='.05'>
+        <xacro:inertial_cylinder mass='0.1' length='.04' radius='.05'>
             <origin xyz='0 0 0' rpy='0 0 0'/>
         </xacro:inertial_cylinder>
@@ -127,5 +127,5 @@
             </geometry>
         </collision>
-        <xacro:inertial_cylinder mass='.1' length='.04' radius='.05'>
+        <xacro:inertial_cylinder mass='0.1' length='.04' radius='.05'>
             <origin xyz='0 0 0' rpy='0 0 0'/>
         </xacro:inertial_cylinder>
