Commit message: change

File: description/lidar.xacro (robot description, xacro)
@@ -5,20 +5,20 @@
         <child link="laser_frame"/>
         <origin xyz="0.1 0.0 0.175" rpy="0.0 0.0 0.0"/>
-        <link name='laser_frame'>
-            <visual>
-                <geometry>
-                    <cylinder radius='0.05' length='0.04'/>
-                </geometry>
-                <material name='red'/>
-            </visual>
-            <collision>
-                <geometry>
-                    <cylinder radius='0.05' length='0.04'/>
-                </geometry>
-            </collision>
-            <xacro:inertial_cylinder mass='0.1' length='.04' radius='.05'>
-                <origin xyz='0 0 0' rpy='0 0 0'/>
-            </xacro:inertial_cylinder>
-        </link>
     </joint>
+    <link name='laser_frame'>
+        <visual>
+            <geometry>
+                <cylinder radius='0.05' length='0.04'/>
+            </geometry>
+            <material name='red'/>
+        </visual>
+        <collision>
+            <geometry>
+                <cylinder radius='0.05' length='0.04'/>
+            </geometry>
+        </collision>
+        <xacro:inertial_cylinder mass='0.1' length='.04' radius='.05'>
+            <origin xyz='0 0 0' rpy='0 0 0'/>
+        </xacro:inertial_cylinder>
+    </link>
 </robot>

Commit message: complete Lidar simulation in Gazebo

File: description/lidar.xacro (robot description, xacro)
@@ -22,3 +22,33 @@
         </xacro:inertial_cylinder>
     </link>
+    <gazebo reference ='laser_frame'>
+        <material>Gazebo/Red</material>
+        <sensor name='laser' type='ray'>
+            <pose> 0 0 0 0 0 0 </pose>
+            <visualize>true</visualize>
+            <update_rate>10</update_rate>
+            <ray>
+                <scan>
+                    <horizontal>
+                        <samples>360</samples>
+                        <resolution>1</resolution>
+                        <min_angle>-3.14</min_angle>
+                        <max_angle>3.14</max_angle>
+                    </horizontal>
+                </scan>
+                <range>
+                    <min>0.3</min>
+                    <max>12</max>
+                    <resolution>0.01</resolution>
+                </range>
+            </ray>
+            <plugin name='laser_controller' filename='libgazebo_ros_ray_sensor.so'>
+                <ros>
+                    <argument>~/out:=scan</argument>
+                </ros>
+                <output_type>sensor_msgs/LaserScan</output_type>
+                <frame_name>laser_frame</frame_name>
+            </plugin>
+        </sensor>
+    </gazebo>
 </robot>
